File: TMC429-Breakout.kicad_sch (KiCad schematic)
At the start: 19 parts, among them U1 TMC429-LI, U2 TMC2130_STEPPER_MOTOR_DRIVER_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, U3 TMC2130_STEPPER_MOTOR_DRIVER_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, U4 TMC2130_STEPPER_MOTOR_DRIVER_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, Y1 CB3LV-3C-32

Commit message: Interim commit
Parts:
- added C18: 0.1uF, symbol Device:C
- added TP1, TP10, TP11, TP12, TP13, TP2, TP3, TP4, TP5, TP6, TP7, TP8, TP9: TestPoint, symbol Connector:TestPoint
- C10, C11, C12: value C_Polarized -> 100uF 35V
Connections:
- net D1: now also TP3.1
- net D2: now also TP5.1
- net D3: now also TP7.1
- net S1: now also TP2.1
- net S2: now also TP4.1
- net S3: now also TP6.1
- net SCLK: now also TP9.1
- net SDI: now also TP8.1
- net SDO: now also TP10.1
- net ~{CS_1}: now also TP11.1
- net ~{CS_2}: now also TP12.1
- net ~{CS_3}: now also TP13.1
